File: ByteDisplay/ByteDisplay.kicad_pcb (KiCad board)
At the start: 2 copper layers, 23.4 x 20.3 mm, 22 parts, among them J1 Conn_01x08_Pin, J2 Conn_01x01_Socket, J3 Conn_01x01_Socket, J4 Conn_01x01_Socket, U1 74HCT573

Commit message: Add pullup resistors to ClockGen and ByteHex
Other:
- board text added: "This work is licensed under the Creative Commons Attribute-ShareAlike 4.0 International License. To view a copy of this license, visit http://creativecommons.org/license/by-sa/4.0/ or send a letter to Creative Commons, PO Box 1866, Mountain View, CA 94042, USA."
Changed lines of the file:
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@@
   )
   (paper "A4")
+  (title_block
+    (title "ByteDisplay")
+    (comment 1 "By Tube Time")
+  )
   (layers
     (0 "F.Cu" signal)
@@
     (effects (font (size 1.016 1.016) (thickness 0.1524)) (justify left bottom))
   )
+  (gr_text "This work is licensed under the Creative Commons\nAttribute-ShareAlike 4.0 International License.\nTo view a copy of this license, visit\nhttp://creativecommons.org/license/by-sa/4.0/\nor send a letter to Creative Commons, PO Box 1866,\nMountain View, CA 94042, USA." (at 119.9 181.4) (layer "Dwgs.User")
+    (effects (font (size 1.27 1.27) (thickness 0.254)) (justify left))
+  )
   (dimension (type aligned) (layer "Dwgs.User")
