File: ByteHex/ByteHex.kicad_sch (KiCad schematic)
At the start: 18 parts, among them J1 Conn_01x08_Pin, J2 Conn_01x01_Socket, J3 Conn_01x01_Socket, J4 Conn_01x01_Socket, J5 ISP, SW4 SW_DIP_x04, U1 ATmega328PB-M

Commit message: Add pullup resistors to ClockGen and ByteHex
Parts:
- added R10: 4.7K, Passive:RESC2012X55, symbol Device:R_Small_US
- SW4: value SW_DIP_x04 -> CONFIG; Mouser CHS-04A -> 229-CHS-04A
- U1: Mouser (none) -> 556-ATMEGA328PB-MU
Connections:
- net VCC: now also R10.1
- net at SW4.8, U1.7 (XTAL1/PB6): now also R10.2
Other:
- note added: "By Tube Time"
- note added: "ByteHex"
- note added: "This work is licensed under the Creative Commons Attribute-ShareAlike 4.0 International License. To view a copy of this license, visit http://creativecommons.org/license/by-sa/4.0/ or send a letter to Creative Commons, PO Box 1866, Mountain View, CA 94042, USA."
- note removed: "Use pin header with .024" instead of 0.026" square pins"
Changed lines of the file:
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@@
 (kicad_sch (version 20230121) (generator eeschema)
   (paper "A4")
+  (junction (at 85.09 82.55) (diameter 0) (color 0 0 0 0)
+  )
   (junction (at 63.5 85.09) (diameter 0) (color 0 0 0 0)
   )
@@
     (stroke (width 0) (type default))
   )
-  (wire (pts (xy 99.06 82.55) (xy 81.28 82.55))
+  (wire (pts (xy 99.06 82.55) (xy 85.09 82.55))
     (stroke (width 0) (type default))
   )
@@
     (stroke (width 0) (type default))
   )
+  (wire (pts (xy 85.09 82.55) (xy 81.28 82.55))
+    (stroke (width 0) (type default))
+  )
   (wire (pts (xy 199.39 44.45) (xy 199.39 50.8))
     (stroke (width 0) (type default))
@@
     (stroke (width 0) (type default))
   )
+  (wire (pts (xy 85.09 80.01) (xy 85.09 82.55))
+    (stroke (width 0) (type default))
+  )
   (wire (pts (xy 63.5 87.63) (xy 63.5 85.09))
     (stroke (width 0) (type default))
@@
     (stroke (width 0) (type default))
   )
-  (text "Use pin header with .024\" instead of 0.026\" square pins"
-    (at 36.83 54.61 0)
-    (effects (font (size 1.27 1.27)) (justify left bottom))
+  (text "This work is licensed under the Creative Commons\nAttribute-ShareAlike 4.0 International License.\nTo view a copy of this license, visit\nhttp://creativecommons.org/license/by-sa/4.0/\nor send a letter to Creative Commons, PO Box 1866,\nMountain View, CA 94042, USA."
+    (at 67.31 190.5 0)
+    (effects (font (size 2.54 2.54)) (justify left bottom))
+  )
+  (text "ByteHex" (at 179.07 173.99 0)
+    (effects (font (size 5.08 5.08)) (justify left bottom))
+  )
+  (text "By Tube Time" (at 180.34 179.07 0)
+    (effects (font (size 2.54 2.54)) (justify left bottom))
   )
   (label "LEDD" (at 177.8 76.2 0) (fields_autoplaced)
@@
     )
     (property "Datasheet" "http://ww1.microchip.com/downloads/en/DeviceDoc/40001906C.pdf" (at 123.19 88.9 0)
+      (effects (font (size 1.27 1.27)) hide)
+    )
+    (property "Mouser" "556-ATMEGA328PB-MU" (at 123.19 88.9 0)
       (effects (font (size 1.27 1.27)) hide)
     )
@@
     )
   )
+  (symbol (lib_id "Device:R_Small_US") (at 85.09 77.47 0) (unit 1)
+    (in_bom yes) (on_board yes) (dnp no) (fields_autoplaced)
+    (property "Reference" "R10" (at 87.63 76.2 0)
+      (effects (font (size 1.27 1.27)) (justify left))
+    )
+    (property "Value" "4.7K" (at 87.63 78.74 0)
+      (effects (font (size 1.27 1.27)) (justify left))
+    )
+    (property "Footprint" "Passive:RESC2012X55" (at 85.09 77.47 0)
+      (effects (font (size 1.27 1.27)) hide)
+    )
+    (property "Datasheet" "~" (at 85.09 77.47 0)
+      (effects (font (size 1.27 1.27)) hide)
+    )
+    (pin "1")
+    (pin "2")
+    (instances
+      (project "ByteHex"
+        (path "/0f695af6-12c5-4431-9904-a6d8e7f13b93"
+          (reference "R10") (unit 1)
+        )
+      )
+    )
+  )
   (symbol (lib_id "Connector_Generic:Conn_02x03_Odd_Even") (at 185.42 53.34 0) (unit 1)
     (in_bom yes) (on_board yes) (dnp no) (fields_autoplaced)
@@
       (effects (font (size 1.27 1.27)))
     )
-    (property "Value" "SW_DIP_x04" (at 73.66 77.47 0)
+    (property "Value" "CONFIG" (at 73.66 77.47 0)
       (effects (font (size 1.27 1.27)))
     )
@@
       (effects (font (size 1.27 1.27)) hide)
     )
-    (property "Mouser" "CHS-04A" (at 73.66 87.63 0)
+    (property "Mouser" "229-CHS-04A" (at 73.66 87.63 0)
       (effects (font (size 1.27 1.27)) hide)
     )
@@
         )
       )
+    )
+  )
+  (symbol (lib_id "power:VCC") (at 85.09 74.93 0) (unit 1)
+    (in_bom yes) (on_board yes) (dnp no) (fields_autoplaced)
+    (property "Reference" "#PWR05" (at 85.09 78.74 0)
+      (effects (font (size 1.27 1.27)) hide)
+    )
+    (property "Value" "VCC" (at 85.09 69.85 0)
+      (effects (font (size 1.27 1.27)))
+    )
+    (property "Footprint" "" (at 85.09 74.93 0)
+      (effects (font (size 1.27 1.27)) hide)
+    )
+    (property "Datasheet" "" (at 85.09 74.93 0)
+      (effects (font (size 1.27 1.27)) hide)
+    )
+    (pin "1")
+    (instances
+      (project "ByteHex"
+        (path "/0f695af6-12c5-4431-9904-a6d8e7f13b93"
+          (reference "#PWR05") (unit 1)
+        )
+      )
