File: ClockGen/ClockGen.kicad_pcb (KiCad board)
At the start: 2 copper layers, 32.1 x 20.3 mm, 22 parts, among them J1 Conn_01x08_Pin, J5 ISP, Q1 2N7002, SW1 RANGE, U1 ATmega328PB-M

Commit message: Add pullup resistors to ClockGen and ByteHex
Parts:
- added R1: 4.7K, Passive:RESC2012X55, B.Cu at (147.3, 115.3)
- added R14: 4.7K, Passive:RESC2012X55, B.Cu at (149.4, 115.3)
- Q1: value 2N7002 -> DMN2053UQ-13
Routing:
- net Net-(U1-XTAL2/PB7): track 15.2 -> 26.4 mm, vias 1 -> 2
- net VCC: track 63.2 -> 66.8 mm
- net Net-(U1-XTAL1/PB6): track 20.3 -> 23.8 mm
- net Net-(U1-AREF): track 11.3 -> 12.0 mm
Other:
- board text added: "This work is licensed under the Creative Commons Attribute-ShareAlike 4.0 International License. To view a copy of this license, visit http://creativecommons.org/license/by-sa/4.0/ or send a letter to Creative Commons, PO Box 1866, Mountain View, CA 94042, USA."
