File: ClockGen/ClockGen.kicad_sch (KiCad schematic)
At the start: 22 parts, among them J1 Conn_01x08_Pin, J5 ISP, Q1 2N7002, SW1 RANGE, U1 ATmega328PB-M

Commit message: Add pullup resistors to ClockGen and ByteHex
Parts:
- added R1, R14: 4.7K, Passive:RESC2012X55, symbol Device:R_Small_US
- D1: Mouser (none) -> 859-LTD-2601G-11
- Q1: value 2N7002 -> DMN2053UQ-13
- RV1, RV2: Mouser (none) -> 594-63P103T7
- U1: Mouser (none) -> 556-ATMEGA328PB-MU
Connections:
- net VCC: now also R1.1, R14.1
- net at SW1.0, U1.7 (XTAL1/PB6): now also R1.2
- net at SW1.1, U1.8 (XTAL2/PB7): now also R14.2
Other:
- note added: "By Tube Time"
- note added: "ClockGen"
- note added: "Potentiometers: You can also use https://www.sparkfun.com/products/9806"
- note added: "This work is licensed under the Creative Commons Attribute-ShareAlike 4.0 International License. To view a copy of this license, visit http://creativecommons.org/license/by-sa/4.0/ or send a letter to Creative Commons, PO Box 1866, Mountain View, CA 94042, USA."
- note removed: "TODO: low Vth FET"
- note removed: "Use bandgap reference on ADC to measure VCC for supply monitor"
- note removed: "pots: use 594-63P103T7, make sure it works with https://www.sparkfun.com/products/9806 range: use 774-220ADC04 or 774-220ADC16."
Changed lines of the file:
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@@
   (junction (at 123.19 49.53) (diameter 0) (color 0 0 0 0)
   )
+  (junction (at 80.01 80.01) (diameter 0) (color 0 0 0 0)
+  )
+  (junction (at 88.9 82.55) (diameter 0) (color 0 0 0 0)
+  )
   (junction (at 199.39 55.88) (diameter 0) (color 0 0 0 0)
   )
@@
     (stroke (width 0) (type default))
   )
+  (wire (pts (xy 80.01 80.01) (xy 96.52 80.01))
+    (stroke (width 0) (type default))
+  )
   (wire (pts (xy 138.43 66.04) (xy 158.75 66.04))
     (stroke (width 0) (type default))
@@
     (stroke (width 0) (type default))
   )
-  (wire (pts (xy 76.2 80.01) (xy 96.52 80.01))
+  (wire (pts (xy 76.2 80.01) (xy 80.01 80.01))
     (stroke (width 0) (type default))
   )
@@
     (stroke (width 0) (type default))
   )
-  (wire (pts (xy 138.43 111.76) (xy 163.83 111.76))
+  (wire (pts (xy 88.9 82.55) (xy 99.06 82.55))
     (stroke (width 0) (type default))
   )
@@
     (stroke (width 0) (type default))
   )
-  (wire (pts (xy 210.82 133.35) (xy 223.52 133.35))
-    (stroke (width 0) (type default))
-  )
   (wire (pts (xy 68.58 104.14) (xy 93.98 104.14))
     (stroke (width 0) (type default))
@@
     (stroke (width 0) (type default))
   )
-  (wire (pts (xy 138.43 119.38) (xy 163.83 119.38))
-    (stroke (width 0) (type default))
-  )
   (wire (pts (xy 63.5 82.55) (xy 66.04 82.55))
     (stroke (width 0) (type default))
@@
     (stroke (width 0) (type default))
   )
-  (wire (pts (xy 76.2 82.55) (xy 99.06 82.55))
+  (wire (pts (xy 80.01 78.74) (xy 80.01 80.01))
+    (stroke (width 0) (type default))
+  )
+  (wire (pts (xy 76.2 82.55) (xy 88.9 82.55))
     (stroke (width 0) (type default))
   )
@@
     (stroke (width 0) (type default))
   )
-  (wire (pts (xy 138.43 116.84) (xy 163.83 116.84))
-    (stroke (width 0) (type default))
-  )
   (wire (pts (xy 123.19 48.26) (xy 123.19 49.53))
     (stroke (width 0) (type default))
@@
     (stroke (width 0) (type default))
   )
-  (wire (pts (xy 138.43 114.3) (xy 163.83 114.3))
-    (stroke (width 0) (type default))
-  )
   (wire (pts (xy 184.15 73.66) (xy 177.8 73.66))
     (stroke (width 0) (type default))
@@
     (stroke (width 0) (type default))
   )
+  (wire (pts (xy 88.9 78.74) (xy 88.9 82.55))
+    (stroke (width 0) (type default))
+  )
   (wire (pts (xy 138.43 81.28) (xy 147.32 81.28))
     (stroke (width 0) (type default))
@@
     (stroke (width 0) (type default))
   )
-  (text_box "TODO:\n* Ranges? 1-100Hz, 100-10KHz, 10KHz-100KHz, 100KHz-1MHz (?)"
-    (at 16.51 17.78 0) (size 57.15 49.53)
-    (stroke (width 0) (type default))
-    (fill (type none))
-    (effects (font (size 1.27 1.27)) (justify left top))
-  )
-  (text "pots: use 594-63P103T7, make sure it works with https://www.sparkfun.com/products/9806\nrange: use 774-220ADC04 or 774-220ADC16.\n"
+  (text "This work is licensed under the Creative Commons\nAttribute-ShareAlike 4.0 International License.\nTo view a copy of this license, visit\nhttp://creativecommons.org/license/by-sa/4.0/\nor send a letter to Creative Commons, PO Box 1866,\nMountain View, CA 94042, USA."
+    (at 67.31 190.5 0)
+    (effects (font (size 2.54 2.54)) (justify left bottom))
+  )
+  (text "Potentiometers: You can also use https://www.sparkfun.com/products/9806\n"
     (at 24.13 142.24 0)
     (effects (font (size 1.27 1.27)) (justify left bottom))
   )
-  (text "TODO: low Vth FET" (at 184.15 149.86 0)
-    (effects (font (size 1.27 1.27)) (justify left bottom))
-  )
-  (text "Use bandgap reference on ADC to measure VCC for supply monitor"
-    (at 113.03 158.75 0)
-    (effects (font (size 1.27 1.27)) (justify left bottom))
-  )
   (text "OC3A" (at 125.73 102.87 0)
     (effects (font (size 1.27 1.27)) (justify left bottom))
   )
+  (text "ClockGen" (at 179.07 173.99 0)
+    (effects (font (size 5.08 5.08)) (justify left bottom))
+  )
+  (text "By Tube Time" (at 180.34 179.07 0)
+    (effects (font (size 2.54 2.54)) (justify left bottom))
+  )
   (label "~{RESETOUT}" (at 210.82 130.81 0) (fields_autoplaced)
     (effects (font (size 1.27 1.27)) (justify left bottom))
@@
       (effects (font (size 1.27 1.27)) hide)
     )
+    (property "Mouser" "594-63P103T7" (at 64.77 104.14 0)
+      (effects (font (size 1.27 1.27)) hide)
+    )
     (pin "1")
     (pin "2")
@@
         (path "/0f695af6-12c5-4431-9904-a6d8e7f13b93"
           (reference "#PWR04") (unit 1)
+        )
+      )
+    )
+  )
+  (symbol (lib_id "Device:R_Small_US") (at 88.9 76.2 0) (unit 1)
+    (in_bom yes) (on_board yes) (dnp no) (fields_autoplaced)
+    (property "Reference" "R14" (at 91.44 74.93 0)
+      (effects (font (size 1.27 1.27)) (justify left))
+    )
+    (property "Value" "4.7K" (at 91.44 77.47 0)
+      (effects (font (size 1.27 1.27)) (justify left))
+    )
+    (property "Footprint" "Passive:RESC2012X55" (at 88.9 76.2 0)
+      (effects (font (size 1.27 1.27)) hide)
+    )
+    (property "Datasheet" "~" (at 88.9 76.2 0)
+      (effects (font (size 1.27 1.27)) hide)
+    )
+    (pin "1")
+    (pin "2")
+    (instances
+      (project "ClockGen"
+        (path "/0f695af6-12c5-4431-9904-a6d8e7f13b93"
+          (reference "R14") (unit 1)
         )
       )
@@
     )
     (property "Datasheet" "http://ww1.microchip.com/downloads/en/DeviceDoc/40001906C.pdf" (at 123.19 88.9 0)
+      (effects (font (size 1.27 1.27)) hide)
+    )
+    (property "Mouser" "556-ATMEGA328PB-MU" (at 123.19 88.9 0)
       (effects (font (size 1.27 1.27)) hide)
     )
@@
       (effects (font (size 1.27 1.27)) hide)
     )
+    (property "Mouser" "859-LTD-2601G-11" (at 198.12 66.04 0)
+      (effects (font (size 1.27 1.27)) hide)
+    )
     (pin "1")
     (pin "10")
@@
       (effects (font (size 1.27 1.27)) hide)
     )
+    (property "Mouser" "594-63P103T7" (at 64.77 121.92 0)
+      (effects (font (size 1.27 1.27)) hide)
+    )
     (pin "1")
     (pin "2")
@@
         (path "/0f695af6-12c5-4431-9904-a6d8e7f13b93"
           (reference "RV1") (unit 1)
+        )
+      )
+    )
+  )
+  (symbol (lib_id "power:VCC") (at 88.9 73.66 0) (unit 1)
+    (in_bom yes) (on_board yes) (dnp no) (fields_autoplaced)
+    (property "Reference" "#PWR016" (at 88.9 77.47 0)
+      (effects (font (size 1.27 1.27)) hide)
+    )
+    (property "Value" "VCC" (at 88.9 68.58 0)
+      (effects (font (size 1.27 1.27)))
+    )
+    (property "Footprint" "" (at 88.9 73.66 0)
+      (effects (font (size 1.27 1.27)) hide)
+    )
+    (property "Datasheet" "" (at 88.9 73.66 0)
+      (effects (font (size 1.27 1.27)) hide)
+    )
+    (pin "1")
+    (instances
+      (project "ClockGen"
+        (path "/0f695af6-12c5-4431-9904-a6d8e7f13b93"
+          (reference "#PWR016") (unit 1)
         )
       )
@@
       (effects (font (size 1.27 1.27)) (justify left))
     )
-    (property "Value" "2N7002" (at 195.58 144.78 0)
+    (property "Value" "DMN2053UQ-13" (at 195.58 144.78 0)
       (effects (font (size 1.27 1.27)) (justify left))
     )
@@
         )
       )
+    )
+  )
+  (symbol (lib_id "Device:R_Small_US") (at 80.01 76.2 0) (unit 1)
+    (in_bom yes) (on_board yes) (dnp no) (fields_autoplaced)
+    (property "Reference" "R1" (at 82.55 74.93 0)
+      (effects (font (size 1.27 1.27)) (justify left))
+    )
+    (property "Value" "4.7K" (at 82.55 77.47 0)
+      (effects (font (size 1.27 1.27)) (justify left))
+    )
+    (property "Footprint" "Passive:RESC2012X55" (at 80.01 76.2 0)
+      (effects (font (size 1.27 1.27)) hide)
+    )
+    (property "Datasheet" "~" (at 80.01 76.2 0)
+      (effects (font (size 1.27 1.27)) hide)
+    )
+    (pin "1")
+    (pin "2")
+    (instances
+      (project "ClockGen"
+        (path "/0f695af6-12c5-4431-9904-a6d8e7f13b93"
+          (reference "R1") (unit 1)
+        )
+      )
+    )
+  )
+  (symbol (lib_id "power:VCC") (at 80.01 73.66 0) (unit 1)
+    (in_bom yes) (on_board yes) (dnp no) (fields_autoplaced)
+    (property "Reference" "#PWR015" (at 80.01 77.47 0)
+      (effects (font (size 1.27 1.27)) hide)
+    )
+    (property "Value" "VCC" (at 80.01 68.58 0)
+      (effects (font (size 1.27 1.27)))
+    )
+    (property "Footprint" "" (at 80.01 73.66 0)
+      (effects (font (size 1.27 1.27)) hide)
+    )
+    (property "Datasheet" "" (at 80.01 73.66 0)
+      (effects (font (size 1.27 1.27)) hide)
+    )
+    (pin "1")
+    (instances
+      (project "ClockGen"
+        (path "/0f695af6-12c5-4431-9904-a6d8e7f13b93"
+          (reference "#PWR015") (unit 1)
+        )
+      )
